Commit message: refactor: migrate arctos control to topic-based ROS2 control plugin

File: src/arctos_description/urdf/hardware/ros2_control.xacro (robot description, xacro)
@@ -6,63 +6,8 @@
     <ros2_control name="${name}" type="system">
       <hardware>
-                <plugin>arctos_hardware_interface/ArctosMKSHardwareInterface</plugin>
-                <param name="motor_can_interface">can0</param>
-                <param name="polling_frequency_hz">30</param>
-                <param name="mks_inter_request_delay_us">500</param>
-        <!-- Motor configuration parameters -->
-        <!-- X_joint -->
-        <param name="motors.X_joint.motor_id">1</param>
-        <param name="motors.X_joint.gear_ratio">13.5</param>
-        <param name="motors.X_joint.inverted">false</param>
-        <param name="motors.X_joint.hardware_type">MKS_57D</param>
-        <param name="motors.X_joint.working_current">2400</param>
-        <param name="motors.X_joint.holding_current">70</param>
-        <param name="motors.X_joint.limit_remap_enabled">false</param>
-        <param name="motors.X_joint.work_mode">5</param>
-        <!-- Y_joint -->
-        <param name="motors.Y_joint.motor_id">2</param>
-        <param name="motors.Y_joint.gear_ratio">150.0</param>
-        <param name="motors.Y_joint.inverted">true</param>
-        <param name="motors.Y_joint.hardware_type">MKS_57D</param>
-        <param name="motors.Y_joint.working_current">2400</param>
-        <param name="motors.Y_joint.holding_current">70</param>
-        <param name="motors.Y_joint.limit_remap_enabled">false</param>
-        <param name="motors.Y_joint.work_mode">5</param>
-        <!-- Z_joint -->
-        <param name="motors.Z_joint.motor_id">3</param>
-        <param name="motors.Z_joint.gear_ratio">150.0</param>
-        <param name="motors.Z_joint.inverted">false</param>
-        <param name="motors.Z_joint.hardware_type">MKS_42D</param>
-        <param name="motors.Z_joint.working_current">1800</param>
-        <param name="motors.Z_joint.holding_current">70</param>
-        <param name="motors.Z_joint.limit_remap_enabled">true</param>
-        <param name="motors.Z_joint.work_mode">5</param>
-        <!-- A_joint -->
-        <param name="motors.A_joint.motor_id">4</param>
-        <param name="motors.A_joint.gear_ratio">48.0</param>
-        <param name="motors.A_joint.inverted">true</param>
-        <param name="motors.A_joint.hardware_type">MKS_42D</param>
-        <param name="motors.A_joint.working_current">1000</param>
-        <param name="motors.A_joint.holding_current">70</param>
-        <param name="motors.A_joint.limit_remap_enabled">true</param>
-        <param name="motors.A_joint.work_mode">5</param>
-        <!-- B_joint -->
-        <param name="motors.B_joint.motor_id">5</param>
-        <param name="motors.B_joint.gear_ratio">27.3375</param>
-        <param name="motors.B_joint.inverted">true</param>
-        <param name="motors.B_joint.hardware_type">MKS_42D</param>
-        <param name="motors.B_joint.working_current">1000</param>
-        <param name="motors.B_joint.holding_current">70</param>
-        <param name="motors.B_joint.limit_remap_enabled">true</param>
-        <param name="motors.B_joint.work_mode">5</param>
-        <!-- C_joint -->
-        <param name="motors.C_joint.motor_id">6</param>
-        <param name="motors.C_joint.gear_ratio">10.0</param>
-        <param name="motors.C_joint.inverted">true</param>
-        <param name="motors.C_joint.hardware_type">MKS_42D</param>
-        <param name="motors.C_joint.working_current">1000</param>
-        <param name="motors.C_joint.holding_current">70</param>
-        <param name="motors.C_joint.limit_remap_enabled">true</param>
-        <param name="motors.C_joint.work_mode">5</param>
+        <plugin>topic_based_ros2_control/TopicBasedSystem</plugin>
+        <param name="joint_commands_topic">/joint_commands_radian</param>
+        <param name="joint_states_topic">/topic_based_joint_states</param>
+        <param name="sum_wrapped_joint_states">true</param>
       </hardware>
       <!-- Interface definitions -->

File: src/arctos_description/urdf/macros/control_macro.xacro (robot description, xacro)
@@ -8,8 +8,5 @@
         <param name="max">${limit_u}</param>
       </command_interface>
-      <command_interface name="velocity">
-        <param name="min">-3.0</param>
-        <param name="max">3.0</param>
-      </command_interface>
+      <command_interface name="velocity"/>
       <state_interface name="position"/>
       <state_interface name="velocity"/>

File: src/arctos_description/urdf/macros/joint_macro.xacro (robot description, xacro)
@@ -13,14 +13,4 @@
       <limit upper="${limit_u}" lower="${limit_l}" effort="${limit_e}" velocity="${limit_v}"/>
     </joint>
-    <!-- generic simple transmission -->
-    <transmission name="transmission_${name}">
-      <type>transmission_interface/SimpleTransmission</type>
-      <joint name="${name}">
-        <hardwareInterface>hardware_interface/PositionJointInterface</hardwareInterface>
-      </joint>
-      <actuator name="${name}_motor">
-        <mechanicalReduction>1.0</mechanicalReduction>
-      </actuator>
-    </transmission>
   </xacro:macro>
 </robot>
