Commit message: docs: clean up repository structure and remove obsolete code
- Removed mks_motor_driver package and scripts/ directory references from AGENTS.md
- Updated documentation to reflect UDP-based hardware interface and FollowJointTrajectory action usage
- Removed arctos_bringup_v2.launch.py and demo.launch.py (consolidated into single bringup launch)
- Cleaned up arctos_bringup CMakeLists.txt: removed unused dependencies and compiler flags
- Removed obsolete template files (.f_tmp, unused controller headers

File: arctos_description/urdf/arctos.urdf.xacro (robot description, xacro)
@@ -1,4 +1,4 @@
 <?xml version="1.0"?>
-<!-- Entry point: include this file to get full Arctos robot description -->
+<!-- Entry point: full Arctos robot description with ros2_control hardware -->
 <robot xmlns:xacro="http://www.ros.org/wiki/xacro" name="arctos">
   <!-- Macro libraries -->
@@ -6,5 +6,4 @@
   <xacro:include filename="$(find arctos_description)/urdf/macros/link_macro.xacro"/>
   <xacro:include filename="$(find arctos_description)/urdf/macros/joint_macro.xacro"/>
-  <xacro:include filename="$(find arctos_description)/urdf/macros/control_macro.xacro"/>
   <!-- Robot sub-assemblies -->
   <xacro:include filename="$(find arctos_description)/urdf/parts/arm_links.xacro"/>
@@ -13,5 +12,4 @@
   <!-- ros2_control hardware definition -->
   <xacro:include filename="$(find arctos_description)/urdf/hardware/ros2_control.xacro"/>
-  <!-- Expose the ros2_control macro so caller can choose the name -->
   <xacro:arctos_ros2_control name="arctos_interface"/>
 </robot>

File: arctos_description/urdf/hardware/ros2_control.xacro (robot description, xacro)
@@ -1,75 +1,55 @@
 <?xml version="1.0"?>
 <robot xmlns:xacro="http://www.ros.org/wiki/xacro" name="arctos">
-  <!-- Provide arctos_ros2_control macro directly (content migrated from old file) -->
-  <xacro:include filename="$(find arctos_description)/urdf/macros/control_macro.xacro"/>
   <xacro:macro name="arctos_ros2_control" params="name">
     <ros2_control name="${name}" type="system">
       <hardware>
-        <plugin>arctos_hardware_interface/STM32StepperInterface</plugin>
+        <plugin>arctos_hardware_interface/STM32HardwareInterface</plugin>
         <param name="stm32_host">192.168.178.159</param>
         <param name="stm32_port">8888</param>
         <!-- Motor configuration parameters -->
         <!-- X_joint -->
-        <param name="motors.X_joint.motor_id">1</param>
         <param name="motors.X_joint.gear_ratio">13.5</param>
         <param name="motors.X_joint.inverted">false</param>
-        <param name="motors.X_joint.hardware_type">MKS_57D</param>
-        <param name="motors.X_joint.working_current">2400</param>
-        <param name="motors.X_joint.holding_current">70</param>
-        <param name="motors.X_joint.limit_remap_enabled">false</param>
-        <param name="motors.X_joint.work_mode">5</param>
         <!-- Y_joint -->
-        <param name="motors.Y_joint.motor_id">2</param>
         <param name="motors.Y_joint.gear_ratio">150.0</param>
         <param name="motors.Y_joint.inverted">false</param>
-        <param name="motors.Y_joint.hardware_type">MKS_57D</param>
-        <param name="motors.Y_joint.working_current">2400</param>
-        <param name="motors.Y_joint.holding_current">70</param>
-        <param name="motors.Y_joint.limit_remap_enabled">false</param>
-        <param name="motors.Y_joint.work_mode">5</param>
         <!-- Z_joint -->
-        <param name="motors.Z_joint.motor_id">3</param>
         <param name="motors.Z_joint.gear_ratio">150.0</param>
         <param name="motors.Z_joint.inverted">false</param>
-        <param name="motors.Z_joint.hardware_type">MKS_42D</param>
-        <param name="motors.Z_joint.working_current">1800</param>
-        <param name="motors.Z_joint.holding_current">70</param>
-        <param name="motors.Z_joint.limit_remap_enabled">true</param>
-        <param name="motors.Z_joint.work_mode">5</param>
         <!-- A_joint -->
-        <param name="motors.A_joint.motor_id">4</param>
         <param name="motors.A_joint.gear_ratio">48.0</param>
         <param name="motors.A_joint.inverted">true</param>
-        <param name="motors.A_joint.hardware_type">MKS_42D</param>
-        <param name="motors.A_joint.working_current">1000</param>
-        <param name="motors.A_joint.holding_current">70</param>
-        <param name="motors.A_joint.limit_remap_enabled">true</param>
-        <param name="motors.A_joint.work_mode">5</param>
         <!-- B_joint -->
-        <param name="motors.B_joint.motor_id">5</param>
         <param name="motors.B_joint.gear_ratio">27.3375</param>
         <param name="motors.B_joint.inverted">false</param>
-        <param name="motors.B_joint.hardware_type">MKS_42D</param>
-        <param name="motors.B_joint.working_current">1000</param>
-        <param name="motors.B_joint.holding_current">70</param>
-        <param name="motors.B_joint.limit_remap_enabled">true</param>
-        <param name="motors.B_joint.work_mode">5</param>
         <!-- C_joint -->
-        <param name="motors.C_joint.motor_id">6</param>
         <param name="motors.C_joint.gear_ratio">10.0</param>
         <param name="motors.C_joint.inverted">true</param>
-        <param name="motors.C_joint.hardware_type">MKS_42D</param>
-        <param name="motors.C_joint.working_current">1000</param>
-        <param name="motors.C_joint.holding_current">70</param>
-        <param name="motors.C_joint.limit_remap_enabled">true</param>
-        <param name="motors.C_joint.work_mode">5</param>
       </hardware>
-      <!-- Interface definitions -->
-      <xacro:arctos_control name="X_joint" limit_u="${pi}" limit_l="${-pi}"/>
-      <xacro:arctos_control name="Y_joint" limit_u="-0.88" limit_l="1.97"/>
-      <xacro:arctos_control name="Z_joint" limit_u="0.65" limit_l="-1.6"/>
-      <xacro:arctos_control name="A_joint" limit_u="${pi}" limit_l="${-pi}"/>
-      <xacro:arctos_control name="B_joint" limit_u="1.55" limit_l="-1.55"/>
-      <xacro:arctos_control name="C_joint" limit_u="${pi}" limit_l="${-pi}"/>
+      <!-- State interfaces (trajectory upload is handled out-of-band by the controller) -->
+      <joint name="X_joint">
+        <state_interface name="position"/>
+        <state_interface name="velocity"/>
+      </joint>
+      <joint name="Y_joint">
+        <state_interface name="position"/>
+        <state_interface name="velocity"/>
+      </joint>
+      <joint name="Z_joint">
+        <state_interface name="position"/>
+        <state_interface name="velocity"/>
+      </joint>
+      <joint name="A_joint">
+        <state_interface name="position"/>
+        <state_interface name="velocity"/>
+      </joint>
+      <joint name="B_joint">
+        <state_interface name="position"/>
+        <state_interface name="velocity"/>
+      </joint>
+      <joint name="C_joint">
+        <state_interface name="position"/>
+        <state_interface name="velocity"/>
+      </joint>
     </ros2_control>
   </xacro:macro>

File: arctos_description/urdf/parts/arm_joints.xacro (robot description, xacro)
@@ -2,5 +2,4 @@
 <robot xmlns:xacro="http://www.ros.org/wiki/xacro" name="arctos">
   <xacro:include filename="$(find arctos_description)/urdf/macros/joint_macro.xacro"/>
-  <xacro:include filename="$(find arctos_description)/urdf/macros/control_macro.xacro"/>
   <!-- World fixed joint -->
   <link name="world"/>
