Commit message: feat: add gripper controller with GripperCommand action support
- Added ArctosGripperController for DS3225MG servo-driven parallel gripper
- Implemented GripperCommand action server with position control and feedback
- Added gripper_controller spawner with conditional launch argument (use_gripper)
- Integrated gripper controller into MoveIt configuration (moveit_controllers.yaml)
- Added Left_jaw_joint position command/state interfaces to ros2_control
- Configured gripper parameters: max_opening_m (

File: arctos_description/urdf/hardware/ros2_control.xacro (robot description, xacro)
@@ -52,4 +52,9 @@
         <state_interface name="velocity"/>
       </joint>
+      <!-- Gripper joint (servo-driven, optional; Right_jaw_joint mimics Left) -->
+      <joint name="Left_jaw_joint">
+        <command_interface name="position"/>
+        <state_interface name="position"/>
+      </joint>
     </ros2_control>
   </xacro:macro>

File: arctos_description/urdf/parts/gripper.xacro (robot description, xacro)
@@ -26,11 +26,16 @@
                       parent="Link_6_1" child="Gripper_1"/>
   <!-- Prismatic jaws -->
-  <xacro:arctos_joint name="Left_jaw_joint" type="fixed"
+  <xacro:arctos_joint name="Left_jaw_joint" type="prismatic"
                       parent="Gripper_1" child="Left_jaw_1"
                       axis_xyz="0 0 -1"
                       limit_u="0.015" limit_l="0" limit_e="1" limit_v="10"/>
-  <xacro:arctos_joint name="Right_jaw_joint" type="fixed"
-                      parent="Gripper_1" child="Right_jaw_1"
-                      axis_xyz="0 0 1"
-                      limit_u="0.015" limit_l="0" limit_e="1" limit_v="10"/>
+  <!-- Right jaw mirrors Left jaw (mimic joint, multiplier=1) -->
+  <joint name="Right_jaw_joint" type="prismatic">
+    <parent link="Gripper_1"/>
+    <child link="Right_jaw_1"/>
+    <origin xyz="0 0 0" rpy="0 0 0"/>
+    <axis xyz="0 0 1"/>
+    <limit upper="0.015" lower="0" effort="1" velocity="10"/>
+    <mimic joint="Left_jaw_joint" multiplier="1.0" offset="0.0"/>
+  </joint>
 </robot>

File: arctos_moveit_config/config/arctos.ros2_control.xacro (robot description, xacro)
@@ -57,11 +57,4 @@
                 </state_interface>
             </joint>
-            <joint name="Right_jaw_joint">
-                <command_interface name="position"/>
-                <command_interface name="velocity"/>
-                <state_interface name="position">
-                  <param name="initial_value">${initial_positions['Right_jaw_joint']}</param>
-                </state_interface>
-            </joint>
         </ros2_control>
     </xacro:macro>
